File: OpenDropV2-ESP201/OpenDropV2-ESP201.sch (KiCad schematic (older format))
At the start: 194 parts, among them J1 DC_JACK, P6 CONN_01X30, Q1 BSS138, Q2 BSS138, Q3 BSS138, Q4 BSS138, Q5 BSS138, SW1 SW_PUSH, SW2 SW_PUSH, SW5 SPST, T1 IRF 840S, U1 MAX1771ESA, U2 HV507, U3 ESP-201, U4 HV507

Commit message: started to clean up schematic
Parts:
- removed C1: 100uF, 35V, Resistors_SMD:R_2512_HandSoldering, symbol CP
- removed C10, C8: 2.2uF, Capacitors_SMD:C_0805, symbol C
- removed C12, C13, C14, C2, C3: 100nF, Capacitors_SMD:C_0805, symbol C
- removed C4: 4u7, 250V, GaudiLabsFootPrints:C_SMD_12mm, symbol CP
- removed C5: 10uF, 25V, Capacitors_SMD:C_1210_HandSoldering, symbol CP
- removed C6: 100nF, 250V, GaudiLabsFootPrints:C100n_250V, symbol C
- removed C7, C9: 1uF, Capacitors_SMD:C_0805, symbol C
- removed D1: ES2F, GaudiLabsFootPrints:DO-214AA, symbol D
- removed FLUXL1, FLUXL10, FLUXL100, FLUXL101, FLUXL102, FLUXL103, FLUXL104, FLUXL105, FLUXL106, FLUXL107, FLUXL108, FLUXL109, FLUXL11, FLUXL110, FLUXL111, FLUXL112, FLUXL113, FLUXL114, FLUXL115, FLUXL116, FLUXL117, FLUXL118, FLUXL119, FLUXL12, FLUXL120, FLUXL121, FLUXL122, FLUXL123, FLUXL124, FLUXL125, FLUXL126, FLUXL127, FLUXL128, FLUXL13, FLUXL14, FLUXL15, FLUXL16, FLUXL17, FLUXL18, FLUXL19, FLUXL2, FLUXL20, FLUXL21, FLUXL22, FLUXL23, FLUXL24, FLUXL25, FLUXL26, FLUXL27, FLUXL28, FLUXL29, FLUXL3, FLUXL30, FLUXL31, FLUXL32, FLUXL33, FLUXL34, FLUXL35, FLUXL36, FLUXL37, FLUXL38, FLUXL39, FLUXL4, FLUXL40, FLUXL41, FLUXL42, FLUXL43, FLUXL44, FLUXL45, FLUXL46, FLUXL47, FLUXL48, FLUXL49, FLUXL5, FLUXL50, FLUXL51, FLUXL52, FLUXL53, FLUXL54, FLUXL55, FLUXL56, FLUXL57, FLUXL58, FLUXL59, FLUXL6, FLUXL60, FLUXL61, FLUXL62, FLUXL63, FLUXL64, FLUXL65, FLUXL66, FLUXL67, FLUXL68, FLUXL69, FLUXL7, FLUXL70, FLUXL71, FLUXL72, FLUXL73, FLUXL74, FLUXL75, FLUXL76, FLUXL77, FLUXL78, FLUXL79, FLUXL8, FLUXL80, FLUXL81, FLUXL82, FLUXL83, FLUXL84, FLUXL85, FLUXL86, FLUXL87, FLUXL88, FLUXL89, FLUXL9, FLUXL90, FLUXL91, FLUXL92, FLUXL93, FLUXL94, FLUXL95, FLUXL96, FLUXL97, FLUXL98, FLUXL99: FX, GaudiLabsFootPrints:FLUXPAD_2_75_4MIL_4_5, symbol FX
- removed J1: DC_JACK, GaudiLabsFootPrints:DC_JACK_SMD, symbol DC_JACK
- removed JS1: JoystickSMD, GaudiLabsFootPrints:JoystickSMD_SKQUSeries, symbol JoystickSMD
- removed L1: 100uH, GaudiLabsFootPrints:Inductor_18.54x15.24, symbol INDUCTOR
- removed LED1, LED8: LED, LEDs:LED-0805, symbol LED
- removed LED2, LED3, LED4, LED5: LED, GaudiLabsFootPrints:LED_SIDE, symbol LED
- removed P6: CONN_01X30, GaudiLabsFootPrints:OLED_SolderPads, symbol CONN_01X30
- removed POT1: 5k Ohm, Potentiometers:Potentiometer_Trimmer-Suntan-TSR-3386P, symbol POT-RESCUE-OpenDropV2
- removed Q1, Q2, Q3, Q4, Q5: BSS138, TO_SOT_Packages_SMD:SOT-23, symbol BSS138
- removed R1: 8k, Resistors_SMD:R_0805, symbol R
- removed R10, R12, R13: 10k, Resistors_SMD:R_0805, symbol R
- removed R11, R14, R18, R19, R20, R21, R22, R23, R24, R25, R8, R9: 10k, symbol R
- removed R15, R16, R17, R7: 10k, GaudiLabsFootPrints:R_0805_HeatPad, symbol R
- removed R2: 1M5, Resistors_SMD:R_2512, symbol R
- removed R3: 390k, Resistors_SMD:R_0805, symbol R
- removed R4, R6: 390, Resistors_SMD:R_0805, symbol R
- removed R5: 10, Resistors_SMD:R_0805, symbol R
- removed RSENSE1: 0R050, Resistors_SMD:R_2010, symbol R
- removed S1: OLED_DISPLAY, GaudiLabsFootPrints:OLED_096_1, symbol OLED_DISPLAY
- removed SP1: SPEAKER, GaudiLabsFootPrints:SMD_PA12_Piezzo, symbol SPEAKER
- removed SW1, SW2: SW_PUSH, GaudiLabsFootPrints:PUSH_BUTTON_SMD, symbol SW_PUSH
- removed SW5: SPST, GaudiLabsFootPrints:Switch_On-On, symbol SPST
- removed T1: IRF 840S, GaudiLabsFootPrints:D2PAK, symbol Q_NMOS_GDS
- removed U1: MAX1771ESA, GaudiLabsFootPrints:SO08, symbol MAX1771ESA
- removed U2, U4: HV507, GaudiLabsFootPrints:PQFP-80_14x20mm_Pitch0.8mm, symbol HV507
- removed U3: ESP-201, symbol ESP-201
Connections:
- net labels removed: +5V, 3.3V, BL, CLK, DI, DISP_RES, DISP_SCL, DISP_SDA, GND, LE, LED_LIGHT, RX_LED, SPK, SW1, SW2, SWCENTER, SWDOWN, SWLEFT, SWRIGHT, SWUP, VIN, V_HV, V_READ_HV
- wire segments 346 -> 0
Other:
- note removed: "65-260VDC"
- note removed: "Controller & WIFI\n"
- note removed: "Display\n"
- note removed: "Fluxl Drivers\n"
- note removed: "High Voltage Generator\n"
- note removed: "LEDs & Switches\n"
- note removed: "Level Shifters\n"
