File: OpenDropV2-ESP201/INDICATORS.sch (KiCad schematic (older format))
At the start: 0 parts

Commit message: worked on lib a little
Parts:
- added SP?: SPEAKER, GaudiLabsFootPrints:SMD_PA12_Piezzo, symbol SPEAKER
Connections:
- new net GND: SP?.1
- new net SPK: SP?.2
Changed lines of the file:
@@
 EELAYER 25 0
 EELAYER END
-$Descr A3 16535 11693
+$Descr A4 11693 8268
 encoding utf-8
-Sheet 1 5
-Title "OpenDrop Version 2"
+Sheet 4 5
+Title ""
 Date ""
-Rev "0.1"
+Rev ""
 Comp ""
 Comment1 ""
@@
 $EndDescr
 $Bitmap
-Pos 11950 6800
+Pos 3400 2900
 Scale 0.000000
 Data
@@
 EndData
 $EndBitmap
-$Sheet
-S 10550 3800 1100 650
-U 5950537C
-F0 "HV_BOOST" 60
-F1 "HV_BOOST.sch" 60
-$EndSheet
-$Sheet
-S 10550 2800 950  700
-U 59505415
-F0 "HV_CONTROLLER" 60
-F1 "HV_CONTROLLER.sch" 60
-$EndSheet
-$Sheet
-S 10600 4800 1050 750
-U 5950AA66
-F0 "INDICATORS" 60
-F1 "INDICATORS.sch" 60
-$EndSheet
-$Sheet
-S 4650 3850 1150 650
-U 5950AAE9
-F0 "ISOLATED SERIAL" 60
-F1 "ISOLATED SERIAL.sch" 60
-$EndSheet
+$Comp
+L SPEAKER SP?
+U 1 1 5950AADC
+P 3000 1700
+F 0 "SP?" H 2900 1950 50  0000 C CNN
+F 1 "SPEAKER" H 2900 1450 50  0000 C CNN
+F 2 "GaudiLabsFootPrints:SMD_PA12_Piezzo" H 3000 1700 60  0001 C CNN
+F 3 "" H 3000 1700 60  0000 C CNN
+	1    3000 1700
+	1    0    0    1
+$EndComp
+Text GLabel 2600 1600 0    60   Input ~ 0
+SPK
+$Comp
+L GND #PWR011
+U 1 1 5950AAE4
+P 2700 2100
+F 0 "#PWR011" H 2700 1850 50  0001 C CNN
+F 1 "GND" H 2700 1950 50  0000 C CNN
+F 2 "" H 2700 2100 60  0000 C CNN
+F 3 "" H 2700 2100 60  0000 C CNN
+	1    2700 2100
+	1    0    0    -1
+$EndComp
+Wire Wire Line
+	2700 1600 2600 1600
+Wire Wire Line
+	2700 1800 2700 2100
 $EndSCHEMATC
